File: Mixed_Signals/mcu_schematic.kicad_sch (KiCad schematic)
At the start: 3 parts, among them J1 Conn_01x02_Pin, U1 ATmega8L-8A

Commit message: cleaned up
Parts:
- J1: footprint (none) -> Connector_PinHeader_2.54mm:PinHeader_1x02_P2.54mm_Vertical
- R1: footprint (none) -> Resistor_SMD:R_0603_1608Metric

Commit message: cleaned up
Parts:
- renumbered J1 to J2, R1 to R4, U1 to U2
Changed lines of the file:
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@@
 		(dnp no)
 		(fields_autoplaced yes)
-		(property "Reference" "U1"
+		(property "Reference" "U2"
 			(at 158.3533 54.61 0)
 			(effects
@@
 			(project "Mixed_Signals"
 				(path "/2e22a617-e9e9-4deb-b0d2-03da1faa5147/2b1b6019-9328-4d81-84dd-1da4a920573e"
-					(reference "U1")
+					(reference "U2")
 					(unit 1)
 				)
@@
 		(dnp no)
 		(fields_autoplaced yes)
-		(property "Reference" "#PWR03"
+		(property "Reference" "#PWR06"
 			(at 153.67 139.7 0)
 			(effects
@@
 			(project "Mixed_Signals"
 				(path "/2e22a617-e9e9-4deb-b0d2-03da1faa5147/2b1b6019-9328-4d81-84dd-1da4a920573e"
-					(reference "#PWR03")
+					(reference "#PWR06")
 					(unit 1)
 				)
@@
 		(dnp no)
 		(fields_autoplaced yes)
-		(property "Reference" "#FLG04"
+		(property "Reference" "#FLG02"
 			(at 151.765 54.61 0)
 			(effects
@@
 			(project "Mixed_Signals"
 				(path "/2e22a617-e9e9-4deb-b0d2-03da1faa5147/2b1b6019-9328-4d81-84dd-1da4a920573e"
-					(reference "#FLG04")
+					(reference "#FLG02")
 					(unit 1)
 				)
@@
 		(dnp no)
 		(fields_autoplaced yes)
-		(property "Reference" "#FLG03"
+		(property "Reference" "#FLG01"
 			(at 118.745 71.12 0)
 			(effects
@@
 			(project "Mixed_Signals"
 				(path "/2e22a617-e9e9-4deb-b0d2-03da1faa5147/2b1b6019-9328-4d81-84dd-1da4a920573e"
-					(reference "#FLG03")
+					(reference "#FLG01")
 					(unit 1)
 				)
@@
 		(dnp no)
 		(fields_autoplaced yes)
-		(property "Reference" "#FLG01"
+		(property "Reference" "#FLG03"
 			(at 156.21 48.895 0)
 			(effects
@@
 			(project ""
 				(path "/2e22a617-e9e9-4deb-b0d2-03da1faa5147/2b1b6019-9328-4d81-84dd-1da4a920573e"
-					(reference "#FLG01")
+					(reference "#FLG03")
 					(unit 1)
 				)
@@
 		(dnp no)
 		(fields_autoplaced yes)
-		(property "Reference" "#PWR02"
+		(property "Reference" "#PWR07"
 			(at 160.02 139.7 0)
 			(effects
@@
 			(project "Mixed_Signals"
 				(path "/2e22a617-e9e9-4deb-b0d2-03da1faa5147/2b1b6019-9328-4d81-84dd-1da4a920573e"
-					(reference "#PWR02")
+					(reference "#PWR07")
 					(unit 1)
 				)
@@
 		(dnp no)
 		(fields_autoplaced yes)
-		(property "Reference" "R1"
+		(property "Reference" "R4"
 			(at 135.89 57.1499 0)
 			(effects
@@
 			(project "Mixed_Signals"
 				(path "/2e22a617-e9e9-4deb-b0d2-03da1faa5147/2b1b6019-9328-4d81-84dd-1da4a920573e"
-					(reference "R1")
+					(reference "R4")
 					(unit 1)
 				)
@@
 		(dnp no)
 		(fields_autoplaced yes)
-		(property "Reference" "#FLG02"
+		(property "Reference" "#FLG04"
 			(at 158.75 130.175 0)
 			(effects
@@
 			(project ""
 				(path "/2e22a617-e9e9-4deb-b0d2-03da1faa5147/2b1b6019-9328-4d81-84dd-1da4a920573e"
-					(reference "#FLG02")
+					(reference "#FLG04")
 					(unit 1)
 				)
@@
 		(dnp no)
 		(fields_autoplaced yes)
-		(property "Reference" "J1"
+		(property "Reference" "J2"
 			(at 116.205 62.23 0)
 			(effects
@@
 			(project "Mixed_Signals"
 				(path "/2e22a617-e9e9-4deb-b0d2-03da1faa5147/2b1b6019-9328-4d81-84dd-1da4a920573e"
-					(reference "J1")
+					(reference "J2")
 					(unit 1)
 				)
@@
 		(dnp no)
 		(fields_autoplaced yes)
-		(property "Reference" "#PWR01"
+		(property "Reference" "#PWR04"
 			(at 120.65 78.74 0)
 			(effects
@@
 			(project "Mixed_Signals"
 				(path "/2e22a617-e9e9-4deb-b0d2-03da1faa5147/2b1b6019-9328-4d81-84dd-1da4a920573e"
-					(reference "#PWR01")
-					(unit 1)
-				)
+					(reference "#PWR04")
+					(unit 1)
+				)
