File: Mixed_Signals/Mixed_Signals.kicad_pcb (KiCad board)
At the start: 2 copper layers, 19 x 28 mm, 12 parts, among them J1 audio connector, J2 Conn_01x02_Pin, U2 ATmega8L-8A

Commit message: modified schematics
Connections:
- R1 pad 2: 5VA -> Net-(U1-+)
Routing:
- net Net-(U1-+): track 13.0 -> 14.4 mm
- net 5VA: track 42.2 -> 41.2 mm
Changed lines of the file:
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@@
 			(layers "F.Cu" "F.Mask" "F.Paste")
 			(roundrect_rratio 0.25)
-			(net 1 "5VA")
+			(net 5 "Net-(U1-+)")
 			(pintype "passive")
 		)
@@
 	)
 	(segment
-		(start 137.735 79.815)
-		(end 139.53 81.61)
+		(start 139.72 81.61)
+		(end 138.745001 81.61)
+		(width 0.1)
+		(layer "F.Cu")
+		(net 1)
+	)
+	(segment
+		(start 138.766164 79.889)
+		(end 140.889 79.889)
+		(width 0.1)
+		(layer "F.Cu")
+		(net 1)
+	)
+	(segment
+		(start 140.889 79.889)
+		(end 142 81)
+		(width 0.1)
+		(layer "F.Cu")
+		(net 1)
+	)
+	(segment
+		(start 138.745001 81.61)
+		(end 138.594 81.458999)
 		(width 0.1)
 		(layer "F.Cu")
@@
 	)
 	(segment
+		(start 139.235 74.1025)
+		(end 139.235 77.180164)
+		(width 0.1)
+		(layer "F.Cu")
+		(net 1)
+	)
+	(segment
+		(start 139.235 77.180164)
+		(end 140.889 78.834164)
+		(width 0.1)
+		(layer "F.Cu")
+		(net 1)
+	)
+	(segment
 		(start 142 82)
 		(end 141.766 82)
@@
 	)
 	(segment
-		(start 139.53 81.61)
-		(end 139.72 81.61)
-		(width 0.1)
-		(layer "F.Cu")
-		(net 1)
-	)
-	(segment
-		(start 136.79 78.87)
-		(end 137.735 79.815)
-		(width 0.1)
-		(layer "F.Cu")
-		(net 1)
-	)
-	(segment
-		(start 141.266 80.481164)
-		(end 140.599836 79.815)
+		(start 142 81)
+		(end 142 82)
+		(width 0.1)
+		(layer "F.Cu")
+		(net 1)
+	)
+	(segment
+		(start 138.594 81.458999)
+		(end 138.594 80.061164)
+		(width 0.1)
+		(layer "F.Cu")
+		(net 1)
+	)
+	(segment
+		(start 138.594 80.061164)
+		(end 138.766164 79.889)
 		(width 0.1)
 		(layer "F.Cu")
@@
 	)
 	(segment
-		(start 140.599836 79.815)
-		(end 137.735 79.815)
-		(width 0.1)
-		(layer "F.Cu")
-		(net 1)
-	)
-	(segment
 		(start 149.5 77.7875)
 		(end 149.5 79)
@@
 	)
 	(segment
-		(start 137.635 78.025)
-		(end 136.79 78.87)
-		(width 0.1)
-		(layer "F.Cu")
-		(net 1)
-	)
-	(segment
 		(start 137.635 74.1025)
 		(end 137.635 73.753188)
@@
 	)
 	(segment
-		(start 137.635 74.1025)
-		(end 137.635 78.025)
+		(start 140.889 78.834164)
+		(end 140.889 79.889)
 		(width 0.1)
 		(layer "F.Cu")
@@
 		(start 136.79 85.017)
 		(end 139.264 87.491)
-		(width 0.1)
-		(layer "F.Cu")
-		(net 1)
-	)
-	(segment
-		(start 141.266 82.5)
-		(end 141.266 80.481164)
 		(width 0.1)
 		(layer "F.Cu")
@@
 	)
 	(segment
+		(start 138.16 78.87)
+		(end 138.17 78.88)
+		(width 0.1)
+		(layer "F.Cu")
+		(net 5)
+	)
+	(segment
 		(start 134.388 78.360812)
 		(end 135.868812 76.88)
@@
 		(width 0.1)
 		(layer "F.Cu")
+		(net 5)
+	)
+	(segment
+		(start 136.79 78.87)
+		(end 138.16 78.87)
+		(width 0.1)
+		(layer "F.Cu")
